Commit message: Change names

File: franka_description/robots/common/franka_hand.xacro (robot description, xacro)
@@ -100,5 +100,5 @@
       </xacro:if>
     </link>
-    <joint name="${arm_id}_finger_joint1" type="prismatic">
+    <joint name="${arm_id}_franka_gripper_finger_joint1" type="prismatic">
       <parent link="${arm_id}_hand" />
       <child link="${arm_id}_leftfinger" />
@@ -108,5 +108,5 @@
       <dynamics damping="0.3" />
     </joint>
-    <joint name="${arm_id}_finger_joint2" type="prismatic">
+    <joint name="${arm_id}_franka_gripper_finger_joint2" type="prismatic">
       <parent link="${arm_id}_hand" />
       <child link="${arm_id}_rightfinger" />
@@ -114,5 +114,5 @@
       <axis xyz="0 -1 0" />
       <limit effort="100" lower="0.0" upper="0.04" velocity="0.2" />
-      <mimic joint="${arm_id}_finger_joint1" />
+      <mimic joint="${arm_id}_franka_gripper_finger_joint1" />
       <dynamics damping="0.3" />
     </joint>

File: franka_description/robots/panda/panda.urdf.xacro (robot description, xacro)
@@ -4,4 +4,5 @@
   <!-- Name for this robot -->
   <xacro:arg name="arm_id" default="panda" />
+  <xacro:arg name="gripper_id" default="$(arg arm_id)_franka_gripper" />
   <!-- Should a franka_gripper be mounted at the flange?" -->
   <xacro:arg name="hand" default="false" />
